File: c64_250407_sram_adapter.kicad_sch (KiCad schematic)
At the start: 19 parts, among them J1 TL_DRAM, J10 B_03, J2 TR_DRAM, J3 BL_DRAM, J4 BR_DRAM, J5 T_01, J6 T_02, J7 T_03, J8 B_01, J9 B_02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

Commit message: Updated PCB to rev.2, adding optional /CAS delay cap
Parts:
- added C4: 100pF-820pF, Capacitor_SMD:C_1206_3216Metric_Pad1.33x1.80mm_HandSolder, symbol Device:C_Small
- added C5: 100pF-820pF, Capacitor_THT:C_Disc_D3.0mm_W2.0mm_P2.50mm, symbol Device:C_Small
Connections:
- net GND: now also C4.2, C5.2
- net ~{CAS}: now also C4.1, C5.1

Commit message: Fixed the silkscreen
Parts:
- C4, C5: value 100pF-820pF -> 82pF-820pF
Changed lines of the file:
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@@
 			)
 		)
-		(property "Value" "100pF-820pF"
+		(property "Value" "82pF-820pF"
 			(at 95.25 97.7962 0)
 			(effects
@@
 			)
 		)
-		(property "Value" "100pF-820pF"
+		(property "Value" "82pF-820pF"
 			(at 76.2 97.7962 0)
 			(effects
